Commit message: update

File: 2.Software/packages/robot_description/urdf/track_cart.urdf (robot description, URDF)
Before this commit: robot track_cart, 7 links, 6 joints
Joints:
- joint camera_joint: origin xyz=0.187658698280417 -0.0010000000000005 0.0983819003855137 rpy=0 0 0 -> xyz=0.187658698280417 -0.0010000000000005 0.6583819003855137 rpy=0 0 0
